File: DSC_motor_controller/CAN.sch (KiCad schematic (older format))
At the start: 3 parts

Commit message: PCB version that will be given to Eric's friend for review
Parts:
- C1: symbol AS0805KKX7R0BB104:AS0805KKX7R0BB104 -> DSC_motor_controller-rescue:AS0805KKX7R0BB104-AS0805KKX7R0BB104
- CAN_TR1: symbol SN65HVD232DR:SN65HVD232DR -> DSC_motor_controller-rescue:SN65HVD232DR-SN65HVD232DR
- RTERM1: symbol ERA3AEB121V:ERA3AEB121V -> DSC_motor_controller-rescue:ERA3AEB121V-ERA3AEB121V
Changed lines of the file:
@@
 EESchema Schematic File Version 4
 LIBS:DSC_motor_controller-cache
-EELAYER 26 0
+EELAYER 29 0
 EELAYER END
 $Descr A4 11693 8268
@@
 $EndDescr
 $Comp
-L SN65HVD232DR:SN65HVD232DR CAN_TR1
+L DSC_motor_controller-rescue:SN65HVD232DR-SN65HVD232DR CAN_TR1
 U 1 1 5D347533
 P 6450 3500
@@
 $EndComp
 $Comp
-L ERA3AEB121V:ERA3AEB121V RTERM1
+L DSC_motor_controller-rescue:ERA3AEB121V-ERA3AEB121V RTERM1
 U 1 1 5D347776
 P 4900 3100
@@
 	5100 3800 4900 3800
 $Comp
-L AS0805KKX7R0BB104:AS0805KKX7R0BB104 C1
+L DSC_motor_controller-rescue:AS0805KKX7R0BB104-AS0805KKX7R0BB104 C1
 U 1 1 5D347B38
 P 7650 3050
