File: DSC_motor_controller/DSC_motor_controller.sch (KiCad schematic (older format))
At the start: 8 parts

Commit message: PCB version that will be given to Eric's friend for review
Parts:
- BUSCNT1, RECV1: symbol SM04B-PASS-TBT(LF)(SN):SM04B-PASS-TBT(LF)(SN) -> DSC_motor_controller-rescue:SM04B-PASS-TBT(LF)(SN)-SM04B-PASS-TBT(LF)(SN)
- C46: footprint CAPC2012X145N -> AS0805KKX7R0BB104:CAPC2012X145N; symbol AS0805KKX7R0BB104:AS0805KKX7R0BB104 -> DSC_motor_controller-rescue:AS0805KKX7R0BB104-AS0805KKX7R0BB104
- D2: symbol LTST-C191KGKT:LTST-C191KGKT -> DSC_motor_controller-rescue:LTST-C191KGKT-LTST-C191KGKT
- D3: symbol LTST-C191KRKT:LTST-C191KRKT -> DSC_motor_controller-rescue:LTST-C191KRKT-LTST-C191KRKT
- R1, R2: symbol RK73H1JTTD1000F:RK73H1JTTD1000F -> DSC_motor_controller-rescue:RK73H1JTTD1000F-RK73H1JTTD1000F
- SWD1: symbol SM05B-PASS-TBT(LF)(SN):SM05B-PASS-TBT(LF)(SN) -> DSC_motor_controller-rescue:SM05B-PASS-TBT(LF)(SN)-SM05B-PASS-TBT(LF)(SN)
Changed lines of the file:
@@
 EESchema Schematic File Version 4
 LIBS:DSC_motor_controller-cache
-EELAYER 26 0
+EELAYER 29 0
 EELAYER END
 $Descr A4 11693 8268
@@
 $EndSheet
 $Comp
-L BLDC_4-cache:PWR_FLAG #FLG0101
+L DSC_motor_controller-rescue:PWR_FLAG-BLDC_4-cache #FLG0101
 U 1 1 5D33E0D2
 P 1750 6900
@@
 $EndComp
 $Comp
-L BLDC_4-cache:PWR_FLAG #FLG0102
+L DSC_motor_controller-rescue:PWR_FLAG-BLDC_4-cache #FLG0102
 U 1 1 5D33E0E2
 P 1750 7100
@@
 $EndComp
 $Comp
-L BLDC_4-cache:PWR_FLAG #FLG0103
+L DSC_motor_controller-rescue:PWR_FLAG-BLDC_4-cache #FLG0103
 U 1 1 5D33E15E
 P 1750 6500
@@
 $EndComp
 $Comp
-L BLDC_4-cache:PWR_FLAG #FLG0104
+L DSC_motor_controller-rescue:PWR_FLAG-BLDC_4-cache #FLG0104
 U 1 1 5D33E164
 P 1750 6700
@@
 SUPPLY
 $Comp
-L BLDC_4-cache:+5V #PWR0101
+L DSC_motor_controller-rescue:+5V-BLDC_4-cache #PWR0101
 U 1 1 5D33F726
 P 2050 6700
@@
 $EndComp
 $Comp
-L LTST-C191KGKT:LTST-C191KGKT D2
+L DSC_motor_controller-rescue:LTST-C191KGKT-LTST-C191KGKT D2
 U 1 1 5D340915
 P 2850 1850
@@
 $EndComp
 $Comp
-L LTST-C191KRKT:LTST-C191KRKT D3
+L DSC_motor_controller-rescue:LTST-C191KRKT-LTST-C191KRKT D3
 U 1 1 5D340BA2
 P 2850 2250
@@
 	1950 2050 1950 2250
 $Comp
-L SM04B-PASS-TBT(LF)(SN):SM04B-PASS-TBT(LF)(SN) RECV1
+L DSC_motor_controller-rescue:SM04B-PASS-TBT(LF)(SN)-SM04B-PASS-TBT(LF)(SN) RECV1
 U 1 1 5D341E7B
 P 1050 2850
@@
 $EndComp
 $Comp
-L SM04B-PASS-TBT(LF)(SN):SM04B-PASS-TBT(LF)(SN) BUSCNT1
+L DSC_motor_controller-rescue:SM04B-PASS-TBT(LF)(SN)-SM04B-PASS-TBT(LF)(SN) BUSCNT1
 U 1 1 5D341F88
 P 1950 3850
@@
 $EndComp
 $Comp
-L SM05B-PASS-TBT(LF)(SN):SM05B-PASS-TBT(LF)(SN) SWD1
+L DSC_motor_controller-rescue:SM05B-PASS-TBT(LF)(SN)-SM05B-PASS-TBT(LF)(SN) SWD1
 U 1 1 5D34214C
 P 1850 5650
@@
 	2050 4950 4200 4950
 $Comp
-L BLDC_4-cache:+5V #PWR0105
+L DSC_motor_controller-rescue:+5V-BLDC_4-cache #PWR0105
 U 1 1 5D343360
 P 1850 3850
@@
 $EndComp
 $Comp
-L BLDC_4-cache:+5V #PWR0109
+L DSC_motor_controller-rescue:+5V-BLDC_4-cache #PWR0109
 U 1 1 5D343BC3
 P 950 2850
@@
 $EndSheet
 $Comp
-L RK73H1JTTD1000F:RK73H1JTTD1000F R1
+L DSC_motor_controller-rescue:RK73H1JTTD1000F-RK73H1JTTD1000F R1
 U 1 1 5D4CBDAD
 P 1950 1850
@@
 $EndComp
 $Comp
-L RK73H1JTTD1000F:RK73H1JTTD1000F R2
+L DSC_motor_controller-rescue:RK73H1JTTD1000F-RK73H1JTTD1000F R2
 U 1 1 5D4CBE5B
 P 1950 2250
@@
 	8450 2650 8750 2650
 $Comp
-L AS0805KKX7R0BB104:AS0805KKX7R0BB104 C46
+L DSC_motor_controller-rescue:AS0805KKX7R0BB104-AS0805KKX7R0BB104 C46
 U 1 1 5D47B463
 P 3200 5100
 F 0 "C46" V 3404 5228 50  0000 L CNN
 F 1 ".1u" V 3495 5228 50  0000 L CNN
-F 2 "CAPC2012X145N" H 3550 5150 50  0001 L CNN
+F 2 "AS0805KKX7R0BB104:CAPC2012X145N" H 3550 5150 50  0001 L CNN
 F 3 "https://mouser.componentsearchengine.com/Datasheets/1/AS0805KKX7R0BB104.pdf" H 3550 5050 50  0001 L CNN
 F 4 "Multilayer Ceramic Capacitors MLCC - SMD/SMT 0.1uF 10% 100V AEC-Q200" H 3550 4950 50  0001 L CNN "Description"
