File: DSC_motor_controller/Motor_Driver.sch (KiCad schematic (older format))
At the start: 36 parts

Commit message: PCB version that will be given to Eric's friend for review
Parts:
- C19: symbol CGA3E2C0G1H682J080AD:CGA3E2C0G1H682J080AD -> DSC_motor_controller-rescue:CGA3E2C0G1H682J080AD-CGA3E2C0G1H682J080AD
- C2, C3: symbol GRM155C81C105ME11J:GRM155C81C105ME11J -> DSC_motor_controller-rescue:GRM155C81C105ME11J-GRM155C81C105ME11J
- C20: symbol C0603C121J5GACTU:C0603C121J5GACTU -> DSC_motor_controller-rescue:C0603C121J5GACTU-C0603C121J5GACTU
- C21: symbol CGA3E2X7R1H223K080AA:CGA3E2X7R1H223K080AA -> DSC_motor_controller-rescue:CGA3E2X7R1H223K080AA-CGA3E2X7R1H223K080AA
- C22, C23, C24, C25, C26: symbol C3216X7R1H225K160AE:C3216X7R1H225K160AE -> DSC_motor_controller-rescue:C3216X7R1H225K160AE-C3216X7R1H225K160AE
- C27, C28, C29: symbol CGA2B3X7R1E224K050BE:CGA2B3X7R1E224K050BE -> DSC_motor_controller-rescue:CGA2B3X7R1E224K050BE-CGA2B3X7R1E224K050BE
- C30: symbol AS0805KKX7R0BB104:AS0805KKX7R0BB104 -> DSC_motor_controller-rescue:AS0805KKX7R0BB104-AS0805KKX7R0BB104
- C31: symbol C0603C153J3GACTU:C0603C153J3GACTU -> DSC_motor_controller-rescue:C0603C153J3GACTU-C0603C153J3GACTU
- C32, C33: symbol CGA6M3X7S2A475K200AB:CGA6M3X7S2A475K200AB -> DSC_motor_controller-rescue:CGA6M3X7S2A475K200AB-CGA6M3X7S2A475K200AB
- C34: symbol 875015119003:875015119003 -> DSC_motor_controller-rescue:875015119003-875015119003
- D1: symbol PMEG6020ER_115:PMEG6020ER,115 -> DSC_motor_controller-rescue:PMEG6020ER,115-PMEG6020ER_115
- DRV1: symbol BLDC_4-cache:DRV8302 -> DSC_motor_controller-rescue:DRV8302-BLDC_4-cache
- L1: symbol SDR0805-220ML:SDR0805-220ML -> DSC_motor_controller-rescue:SDR0805-220ML-SDR0805-220ML
- R16: symbol RK73H1JTTD3301F:RK73H1JTTD3301F -> DSC_motor_controller-rescue:RK73H1JTTD3301F-RK73H1JTTD3301F
- R17: symbol RK73H1JTTD1802F:RK73H1JTTD1802F -> DSC_motor_controller-rescue:RK73H1JTTD1802F-RK73H1JTTD1802F
- R18: symbol RK73H1JTTD1502F:RK73H1JTTD1502F -> DSC_motor_controller-rescue:RK73H1JTTD1502F-RK73H1JTTD1502F
- R19: symbol RK73H1JTTD2203F:RK73H1JTTD2203F -> DSC_motor_controller-rescue:RK73H1JTTD2203F-RK73H1JTTD2203F
- R20: symbol RK73H1JTTD1004F:RK73H1JTTD1004F -> DSC_motor_controller-rescue:RK73H1JTTD1004F-RK73H1JTTD1004F
- R21: symbol RK73H1JTTD1002F:RK73H1JTTD1002F -> DSC_motor_controller-rescue:RK73H1JTTD1002F-RK73H1JTTD1002F
- R22, R23, R24, R25: symbol RK73H1JTTD2201F:RK73H1JTTD2201F -> DSC_motor_controller-rescue:RK73H1JTTD2201F-RK73H1JTTD2201F
- R26, R27, R28, R29: symbol ERJ3EKF3902V:ERJ3EKF3902V -> DSC_motor_controller-rescue:ERJ3EKF3902V-ERJ3EKF3902V
- Reg1: symbol TC2117-3.3VDBTR:TC2117-3.3VDBTR -> DSC_motor_controller-rescue:TC2117-3.3VDBTR-TC2117-3.3VDBTR
Connections:
- wire segments 141 -> 140
Changed lines of the file:
@@
 EESchema Schematic File Version 4
 LIBS:DSC_motor_controller-cache
-EELAYER 26 0
+EELAYER 29 0
 EELAYER END
 $Descr A4 11693 8268
@@
 $EndDescr
 $Comp
-L TC2117-3.3VDBTR:TC2117-3.3VDBTR Reg1
+L DSC_motor_controller-rescue:TC2117-3.3VDBTR-TC2117-3.3VDBTR Reg1
 U 1 1 5D34C356
 P 2850 6800
@@
 $EndComp
 $Comp
-L GRM155C81C105ME11J:GRM155C81C105ME11J C2
+L DSC_motor_controller-rescue:GRM155C81C105ME11J-GRM155C81C105ME11J C2
 U 1 1 5D34C7D9
 P 4400 6800
@@
 $EndComp
 $Comp
-L GRM155C81C105ME11J:GRM155C81C105ME11J C3
+L DSC_motor_controller-rescue:GRM155C81C105ME11J-GRM155C81C105ME11J C3
 U 1 1 5D34C879
 P 2350 7450
@@
 $EndComp
 $Comp
-L BLDC_4-cache:+5V #PWR0126
+L DSC_motor_controller-rescue:+5V-BLDC_4-cache #PWR0126
 U 1 1 5D34CB5D
 P 4400 6800
@@
 NoConn ~ 4150 6900
 $Comp
-L BLDC_4-cache:DRV8302 DRV1
+L DSC_motor_controller-rescue:DRV8302-BLDC_4-cache DRV1
 U 1 1 5D363539
 P 5450 4150
@@
 $EndComp
 $Comp
-L RK73H1JTTD1802F:RK73H1JTTD1802F R17
+L DSC_motor_controller-rescue:RK73H1JTTD1802F-RK73H1JTTD1802F R17
 U 1 1 5D363C64
 P 2650 2850
@@
 $EndComp
 $Comp
-L CGA3E2C0G1H682J080AD:CGA3E2C0G1H682J080AD C19
+L DSC_motor_controller-rescue:CGA3E2C0G1H682J080AD-CGA3E2C0G1H682J080AD C19
 U 1 1 5D363ED7
 P 3500 2000
@@
 $EndComp
 $Comp
-L C0603C121J5GACTU:C0603C121J5GACTU C20
+L DSC_motor_controller-rescue:C0603C121J5GACTU-C0603C121J5GACTU C20
 U 1 1 5D3640D5
 P 3850 2350
@@
 $EndComp
 $Comp
-L RK73H1JTTD1502F:RK73H1JTTD1502F R18
+L DSC_motor_controller-rescue:RK73H1JTTD1502F-RK73H1JTTD1502F R18
 U 1 1 5D364780
 P 3500 2900
@@
 $EndComp
 $Comp
-L RK73H1JTTD2203F:RK73H1JTTD2203F R19
+L DSC_motor_controller-rescue:RK73H1JTTD2203F-RK73H1JTTD2203F R19
 U 1 1 5D3652F1
 P 4250 2350
@@
 $EndComp
 $Comp
-L RK73H1JTTD3301F:RK73H1JTTD3301F R16
+L DSC_motor_controller-rescue:RK73H1JTTD3301F-RK73H1JTTD3301F R16
 U 1 1 5D36586D
 P 2650 2000
@@
 $EndComp
 $Comp
-L BLDC_4-cache:+5V #PWR0130
+L DSC_motor_controller-rescue:+5V-BLDC_4-cache #PWR0130
 U 1 1 5D366631
 P 2300 2750
@@
 NoConn ~ 6250 2900
 $Comp
-L RK73H1JTTD1004F:RK73H1JTTD1004F R20
+L DSC_motor_controller-rescue:RK73H1JTTD1004F-RK73H1JTTD1004F R20
 U 1 1 5D36A842
 P 6450 3500
@@
 $EndComp
 $Comp
-L RK73H1JTTD1002F:RK73H1JTTD1002F R21
+L DSC_motor_controller-rescue:RK73H1JTTD1002F-RK73H1JTTD1002F R21
 U 1 1 5D36BE7E
 P 4200 3400
@@
 	4650 3800 4100 3800
 $Comp
-L CGA3E2X7R1H223K080AA:CGA3E2X7R1H223K080AA C21
+L DSC_motor_controller-rescue:CGA3E2X7R1H223K080AA-CGA3E2X7R1H223K080AA C21
 U 1 1 5D36E996
 P 3800 4150
@@
 	4550 4200 4650 4200
 $Comp
-L C3216X7R1H225K160AE:C3216X7R1H225K160AE C22
+L DSC_motor_controller-rescue:C3216X7R1H225K160AE-C3216X7R1H225K160AE C22
 U 1 1 5D3728B6
 P 4000 5550
@@
 $EndComp
 $Comp
-L C3216X7R1H225K160AE:C3216X7R1H225K160AE C23
+L DSC_motor_controller-rescue:C3216X7R1H225K160AE-C3216X7R1H225K160AE C23
 U 1 1 5D3731EB
 P 3600 5100
@@
 $EndComp
 $Comp
-L C3216X7R1H225K160AE:C3216X7R1H225K160AE C24
+L DSC_motor_controller-rescue:C3216X7R1H225K160AE-C3216X7R1H225K160AE C24
 U 1 1 5D373849
 P 3600 4800
@@
 $EndComp
 $Comp
-L C3216X7R1H225K160AE:C3216X7R1H225K160AE C25
+L DSC_motor_controller-rescue:C3216X7R1H225K160AE-C3216X7R1H225K160AE C25
 U 1 1 5D373EA3
 P 3150 4000
@@
 $EndComp
 $Comp
-L C3216X7R1H225K160AE:C3216X7R1H225K160AE C26
+L DSC_motor_controller-rescue:C3216X7R1H225K160AE-C3216X7R1H225K160AE C26
 U 1 1 5D374535
 P 9100 3350
@@
 PWM_C_L
 Wire Wire Line
-	3600 5000 3600 4800
-Wire Wire Line
 	3600 5100 3600 5000
-Connection ~ 3600 5000
 Wire Wire Line
 	3300 4250 4550 4250
@@
 	4350 4150 3800 4150
 $Comp
-L CGA2B3X7R1E224K050BE:CGA2B3X7R1E224K050BE C29
+L DSC_motor_controller-rescue:CGA2B3X7R1E224K050BE-CGA2B3X7R1E224K050BE C29
 U 1 1 5D383FF6
 P 6600 3700
@@
 $EndComp
 $Comp
-L CGA2B3X7R1E224K050BE:CGA2B3X7R1E224K050BE C28
+L DSC_motor_controller-rescue:CGA2B3X7R1E224K050BE-CGA2B3X7R1E224K050BE C28
 U 1 1 5D3840F8
 P 6600 4100
@@
 $EndComp
 $Comp
-L CGA2B3X7R1E224K050BE:CGA2B3X7R1E224K050BE C27
+L DSC_motor_controller-rescue:CGA2B3X7R1E224K050BE-CGA2B3X7R1E224K050BE C27
 U 1 1 5D384189
 P 6600 4600
@@
 $EndComp
 $Comp
-L AS0805KKX7R0BB104:AS0805KKX7R0BB104 C30
+L DSC_motor_controller-rescue:AS0805KKX7R0BB104-AS0805KKX7R0BB104 C30
 U 1 1 5D38472C
 P 6650 3200
@@
 $EndComp
 $Comp
-L C0603C153J3GACTU:C0603C153J3GACTU C31
+L DSC_motor_controller-rescue:C0603C153J3GACTU-C0603C153J3GACTU C31
 U 1 1 5D38487F
 P 6650 2600
@@
 $EndComp
 $Comp
-L SDR0805-220ML:SDR0805-220ML L1
+L DSC_motor_controller-rescue:SDR0805-220ML-SDR0805-220ML L1
 U 1 1 5D3849DB
 P 8000 3350
@@
 $EndComp
 $Comp
-L PMEG6020ER_115:PMEG6020ER,115 D1
+L DSC_motor_controller-rescue:PMEG6020ER,115-PMEG6020ER_115 D1
 U 1 1 5D385096
 P 7750 3200
@@
 SUPPLY
 $Comp
-L CGA6M3X7S2A475K200AB:CGA6M3X7S2A475K200AB C33
+L DSC_motor_controller-rescue:CGA6M3X7S2A475K200AB-CGA6M3X7S2A475K200AB C33
 U 1 1 5D384454
 P 6500 5650
@@
 	9100 3900 7750 3900
 $Comp
-L 875015119003:875015119003 C34
+L DSC_motor_controller-rescue:875015119003-875015119003 C34
 U 1 1 5D3AF060
 P 9650 3300
+AR Path="/5D3AF060" Ref="C34"  Part="1"
+AR Path="/5D34E5A4/5D3AF060" Ref="C34"  Part="1"
 F 0 "C34" V 9854 3430 50  0000 L CNN
 F 1 "100u" V 9945 3430 50  0000 L CNN
@@
 Connection ~ 6250 3300
 $Comp
-L CGA6M3X7S2A475K200AB:CGA6M3X7S2A475K200AB C32
+L DSC_motor_controller-rescue:CGA6M3X7S2A475K200AB-CGA6M3X7S2A475K200AB C32
 U 1 1 5D3BA05E
 P 7450 2250
@@
 Connection ~ 9650 3900
 $Comp
-L BLDC_4-cache:+5V #PWR0144
+L DSC_motor_controller-rescue:+5V-BLDC_4-cache #PWR0144
 U 1 1 5D3F3151
 P 9650 3000
@@
 	7850 2250 8150 2250
 $Comp
-L ERJ3EKF3902V:ERJ3EKF3902V R29
+L DSC_motor_controller-rescue:ERJ3EKF3902V-ERJ3EKF3902V R29
 U 1 1 5D417FBD
 P 9750 4250
@@
 $EndComp
 $Comp
-L ERJ3EKF3902V:ERJ3EKF3902V R26
+L DSC_motor_controller-rescue:ERJ3EKF3902V-ERJ3EKF3902V R26
 U 1 1 5D41EDD3
 P 9750 4750
@@
 $EndComp
 $Comp
-L ERJ3EKF3902V:ERJ3EKF3902V R27
+L DSC_motor_controller-rescue:ERJ3EKF3902V-ERJ3EKF3902V R27
 U 1 1 5D421F74
 P 9750 5250
@@
 $EndComp
 $Comp
-L ERJ3EKF3902V:ERJ3EKF3902V R28
+L DSC_motor_controller-rescue:ERJ3EKF3902V-ERJ3EKF3902V R28
 U 1 1 5D425119
 P 9750 5750
@@
 $EndComp
 $Comp
-L RK73H1JTTD2201F:RK73H1JTTD2201F R25
+L DSC_motor_controller-rescue:RK73H1JTTD2201F-RK73H1JTTD2201F R25
 U 1 1 5D44D9FA
 P 10450 4450
@@
 $EndComp
 $Comp
-L RK73H1JTTD2201F:RK73H1JTTD2201F R22
+L DSC_motor_controller-rescue:RK73H1JTTD2201F-RK73H1JTTD2201F R22
 U 1 1 5D450BB7
 P 10450 4950
@@
 $EndComp
 $Comp
-L RK73H1JTTD2201F:RK73H1JTTD2201F R23
+L DSC_motor_controller-rescue:RK73H1JTTD2201F-RK73H1JTTD2201F R23
 U 1 1 5D453D66
 P 10450 5450
@@
 $EndComp
 $Comp
-L RK73H1JTTD2201F:RK73H1JTTD2201F R24
+L DSC_motor_controller-rescue:RK73H1JTTD2201F-RK73H1JTTD2201F R24
 U 1 1 5D456F1B
 P 10450 6000
@@
 	4000 5400 4650 5400
 Wire Wire Line
-	3600 5000 4100 5000
-Connection ~ 4100 5000
-Wire Wire Line
-	4100 5000 4650 5000
-Wire Wire Line
 	2850 6050 2850 5000
 Wire Wire Line
@@
 Connection ~ 4000 6050
 Wire Wire Line
-	4100 3800 4100 5000
-Wire Wire Line
 	4650 4000 3150 4000
 Connection ~ 2850 6050
@@
 	4000 6050 4500 6050
 Connection ~ 2850 5000
+Wire Wire Line
+	3600 5000 4650 5000
+Wire Wire Line
+	4100 3800 4100 4800
+Wire Wire Line
+	4100 4800 3600 4800
+$Comp
+L power:GND #PWR0139
+U 1 1 5D50B2C2
+P 4300 5100
+F 0 "#PWR0139" H 4300 4850 50  0001 C CNN
+F 1 "GND" H 4305 4927 50  0000 C CNN
+F 2 "" H 4300 5100 50  0001 C CNN
+F 3 "" H 4300 5100 50  0001 C CNN
+	1    4300 5100
+	1    0    0    -1
+$EndComp
 $EndSCHEMATC
