File: DSC_motor_controller/Motor_controller.sch (KiCad schematic (older format))
At the start: 12 parts

Commit message: PCB version that will be given to Eric's friend for review
Parts:
- C35: symbol GRM155C81C105ME11J:GRM155C81C105ME11J -> DSC_motor_controller-rescue:GRM155C81C105ME11J-GRM155C81C105ME11J
- C36, C37: symbol C3216X7R1H225K160AE:C3216X7R1H225K160AE -> DSC_motor_controller-rescue:C3216X7R1H225K160AE-C3216X7R1H225K160AE
- C38: symbol CGA6M3X7S2A475K200AB:CGA6M3X7S2A475K200AB -> DSC_motor_controller-rescue:CGA6M3X7S2A475K200AB-CGA6M3X7S2A475K200AB
- C39, C40, C41, C42, C43, C44, C45: symbol AS0805KKX7R0BB104:AS0805KKX7R0BB104 -> DSC_motor_controller-rescue:AS0805KKX7R0BB104-AS0805KKX7R0BB104
- DSC1: symbol STM32F765VIT6:STM32F765VIT6 -> DSC_motor_controller-rescue:STM32F765VIT6-STM32F765VIT6
Changed lines of the file:
@@
 EESchema Schematic File Version 4
 LIBS:DSC_motor_controller-cache
-EELAYER 26 0
+EELAYER 29 0
 EELAYER END
 $Descr A4 11693 8268
@@
 $EndDescr
 $Comp
-L STM32F765VIT6:STM32F765VIT6 DSC?
+L DSC_motor_controller-rescue:STM32F765VIT6-STM32F765VIT6 DSC?
 U 1 1 5D33B539
 P 3850 2250
@@
 SWCLK
 $Comp
-L GRM155C81C105ME11J:GRM155C81C105ME11J C35
+L DSC_motor_controller-rescue:GRM155C81C105ME11J-GRM155C81C105ME11J C35
 U 1 1 5D33BFEE
 P 2100 4550
@@
 	2100 4050 2350 4050
 $Comp
-L C3216X7R1H225K160AE:C3216X7R1H225K160AE C37
+L DSC_motor_controller-rescue:C3216X7R1H225K160AE-C3216X7R1H225K160AE C37
 U 1 1 5D33FBF9
 P 8550 2750
@@
 $EndComp
 $Comp
-L C3216X7R1H225K160AE:C3216X7R1H225K160AE C36
+L DSC_motor_controller-rescue:C3216X7R1H225K160AE-C3216X7R1H225K160AE C36
 U 1 1 5D33FC4F
 P 7400 6350
@@
 	6450 5350 6450 5850
 $Comp
-L CGA6M3X7S2A475K200AB:CGA6M3X7S2A475K200AB C38
+L DSC_motor_controller-rescue:CGA6M3X7S2A475K200AB-CGA6M3X7S2A475K200AB C38
 U 1 1 5D341643
 P 1900 2750
@@
 $EndComp
 $Comp
-L AS0805KKX7R0BB104:AS0805KKX7R0BB104 C45
+L DSC_motor_controller-rescue:AS0805KKX7R0BB104-AS0805KKX7R0BB104 C45
 U 1 1 5D341A3F
 P 4200 800
@@
 $EndComp
 $Comp
-L AS0805KKX7R0BB104:AS0805KKX7R0BB104 C44
+L DSC_motor_controller-rescue:AS0805KKX7R0BB104-AS0805KKX7R0BB104 C44
 U 1 1 5D341B54
 P 7750 1850
@@
 $EndComp
 $Comp
-L AS0805KKX7R0BB104:AS0805KKX7R0BB104 C43
+L DSC_motor_controller-rescue:AS0805KKX7R0BB104-AS0805KKX7R0BB104 C43
 U 1 1 5D341BAB
 P 8050 5350
@@
 $EndComp
 $Comp
-L AS0805KKX7R0BB104:AS0805KKX7R0BB104 C40
+L DSC_motor_controller-rescue:AS0805KKX7R0BB104-AS0805KKX7R0BB104 C40
 U 1 1 5D341BDE
 P 2550 2750
@@
 $EndComp
 $Comp
-L AS0805KKX7R0BB104:AS0805KKX7R0BB104 C39
+L DSC_motor_controller-rescue:AS0805KKX7R0BB104-AS0805KKX7R0BB104 C39
 U 1 1 5D341C13
 P 3150 2750
@@
 $EndComp
 $Comp
-L AS0805KKX7R0BB104:AS0805KKX7R0BB104 C41
+L DSC_motor_controller-rescue:AS0805KKX7R0BB104-AS0805KKX7R0BB104 C41
 U 1 1 5D341CBA
 P 2750 4550
@@
 $EndComp
 $Comp
-L AS0805KKX7R0BB104:AS0805KKX7R0BB104 C42
+L DSC_motor_controller-rescue:AS0805KKX7R0BB104-AS0805KKX7R0BB104 C42
 U 1 1 5D341D0D
 P 4500 6650
