File: DSC_motor_controller/Power.sch (KiCad schematic (older format))
At the start: 43 parts, among them P1 PH_A, P2 PH_B, P3 PH_C, P4 SUPPLY, P5 GND, Q1 IRFS7730TRLPBF, Q2 IRFS7730TRLPBF, Q3 IRFS7730TRLPBF, Q4 IRFS7730TRLPBF, Q5 IRFS7730TRLPBF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

Commit message: PCB version that will be given to Eric's friend for review
Parts:
- C10, C11, C12: symbol GCM155R71H472KA37D:GCM155R71H472KA37D -> DSC_motor_controller-rescue:GCM155R71H472KA37D-GCM155R71H472KA37D
- C13, C14, C15, C16: symbol C3216X7R1H225K160AE:C3216X7R1H225K160AE -> DSC_motor_controller-rescue:C3216X7R1H225K160AE-C3216X7R1H225K160AE
- C4, C5, C6, C7, C8, C9: symbol CGA6M3X7S2A475K200AB:CGA6M3X7S2A475K200AB -> DSC_motor_controller-rescue:CGA6M3X7S2A475K200AB-CGA6M3X7S2A475K200AB
- CS1, CS2, CS3: symbol AD8418ABRMZ:AD8418ABRMZ -> DSC_motor_controller-rescue:AD8418ABRMZ-AD8418ABRMZ
- P1, P2, P3, P4, P5: symbol BLDC_4-cache:wire_pad -> DSC_motor_controller-rescue:wire_pad-BLDC_4-cache
- Q1, Q2, Q3, Q4, Q5, Q6: symbol IRFS7730TRLPBF:IRFS7730TRLPBF -> DSC_motor_controller-rescue:IRFS7730TRLPBF-IRFS7730TRLPBF
- R10, R11, R9: symbol WSLP27261L000FEA:WSLP27261L000FEA -> DSC_motor_controller-rescue:WSLP27261L000FEA-WSLP27261L000FEA
- R12, R13, R14: symbol RK73H1JTTD1000F:RK73H1JTTD1000F -> DSC_motor_controller-rescue:RK73H1JTTD1000F-RK73H1JTTD1000F
- R15: symbol RK73H1JTTD1002F:RK73H1JTTD1002F -> DSC_motor_controller-rescue:RK73H1JTTD1002F-RK73H1JTTD1002F
- R3, R4, R5, R6, R7, R8: symbol RK73H1JTTD4R70F:RK73H1JTTD4R70F -> DSC_motor_controller-rescue:RK73H1JTTD4R70F-RK73H1JTTD4R70F
- RTEMP1: symbol NCP18XH103F03RB:NCP18XH103F03RB -> DSC_motor_controller-rescue:NCP18XH103F03RB-NCP18XH103F03RB
Changed lines of the file:
@@
 EESchema Schematic File Version 4
 LIBS:DSC_motor_controller-cache
-EELAYER 26 0
+EELAYER 29 0
 EELAYER END
 $Descr A4 11693 8268
@@
 $EndDescr
 $Comp
-L IRFS7730TRLPBF:IRFS7730TRLPBF Q5
+L DSC_motor_controller-rescue:IRFS7730TRLPBF-IRFS7730TRLPBF Q5
 U 1 1 5D3559AE
 P 9850 1550
@@
 $EndComp
 $Comp
-L CGA6M3X7S2A475K200AB:CGA6M3X7S2A475K200AB C8
+L DSC_motor_controller-rescue:CGA6M3X7S2A475K200AB-CGA6M3X7S2A475K200AB C8
 U 1 1 5D3564BF
 P 10550 2200
@@
 $EndComp
 $Comp
-L CGA6M3X7S2A475K200AB:CGA6M3X7S2A475K200AB C9
+L DSC_motor_controller-rescue:CGA6M3X7S2A475K200AB-CGA6M3X7S2A475K200AB C9
 U 1 1 5D35650A
 P 10850 2200
@@
 $EndComp
 $Comp
-L RK73H1JTTD4R70F:RK73H1JTTD4R70F R7
+L DSC_motor_controller-rescue:RK73H1JTTD4R70F-RK73H1JTTD4R70F R7
 U 1 1 5D356E89
 P 9000 1550
@@
 $EndComp
 $Comp
-L RK73H1JTTD4R70F:RK73H1JTTD4R70F R8
+L DSC_motor_controller-rescue:RK73H1JTTD4R70F-RK73H1JTTD4R70F R8
 U 1 1 5D356EC4
 P 9050 4250
@@
 $EndComp
 $Comp
-L WSLP27261L000FEA:WSLP27261L000FEA R11
+L DSC_motor_controller-rescue:WSLP27261L000FEA-WSLP27261L000FEA R11
 U 1 1 5D3575AC
 P 8450 2000
@@
 $EndComp
 $Comp
-L AD8418ABRMZ:AD8418ABRMZ CS3
+L DSC_motor_controller-rescue:AD8418ABRMZ-AD8418ABRMZ CS3
 U 1 1 5D3579E6
 P 7850 3250
@@
 $EndComp
 $Comp
-L IRFS7730TRLPBF:IRFS7730TRLPBF Q6
+L DSC_motor_controller-rescue:IRFS7730TRLPBF-IRFS7730TRLPBF Q6
 U 1 1 5D35853D
 P 9850 4250
@@
 Connection ~ 9550 3350
 $Comp
-L C3216X7R1H225K160AE:C3216X7R1H225K160AE C15
+L DSC_motor_controller-rescue:C3216X7R1H225K160AE-C3216X7R1H225K160AE C15
 U 1 1 5D35C7FA
 P 8200 3950
@@
 	10150 2000 10150 2300
 $Comp
-L IRFS7730TRLPBF:IRFS7730TRLPBF Q3
+L DSC_motor_controller-rescue:IRFS7730TRLPBF-IRFS7730TRLPBF Q3
 U 1 1 5D36E867
 P 6300 1500
@@
 $EndComp
 $Comp
-L CGA6M3X7S2A475K200AB:CGA6M3X7S2A475K200AB C6
+L DSC_motor_controller-rescue:CGA6M3X7S2A475K200AB-CGA6M3X7S2A475K200AB C6
 U 1 1 5D36E876
 P 7000 2350
@@
 $EndComp
 $Comp
-L CGA6M3X7S2A475K200AB:CGA6M3X7S2A475K200AB C7
+L DSC_motor_controller-rescue:CGA6M3X7S2A475K200AB-CGA6M3X7S2A475K200AB C7
 U 1 1 5D36E885
 P 7250 2350
@@
 $EndComp
 $Comp
-L RK73H1JTTD4R70F:RK73H1JTTD4R70F R5
+L DSC_motor_controller-rescue:RK73H1JTTD4R70F-RK73H1JTTD4R70F R5
 U 1 1 5D36E894
 P 5450 1500
@@
 $EndComp
 $Comp
-L RK73H1JTTD4R70F:RK73H1JTTD4R70F R6
+L DSC_motor_controller-rescue:RK73H1JTTD4R70F-RK73H1JTTD4R70F R6
 U 1 1 5D36E8A3
 P 5500 4200
@@
 $EndComp
 $Comp
-L WSLP27261L000FEA:WSLP27261L000FEA R10
+L DSC_motor_controller-rescue:WSLP27261L000FEA-WSLP27261L000FEA R10
 U 1 1 5D36E8B2
 P 4900 1950
@@
 $EndComp
 $Comp
-L AD8418ABRMZ:AD8418ABRMZ CS2
+L DSC_motor_controller-rescue:AD8418ABRMZ-AD8418ABRMZ CS2
 U 1 1 5D36E8C1
 P 4300 3200
@@
 $EndComp
 $Comp
-L IRFS7730TRLPBF:IRFS7730TRLPBF Q4
+L DSC_motor_controller-rescue:IRFS7730TRLPBF-IRFS7730TRLPBF Q4
 U 1 1 5D36E8D2
 P 6300 4200
@@
 Connection ~ 6000 3300
 $Comp
-L C3216X7R1H225K160AE:C3216X7R1H225K160AE C14
+L DSC_motor_controller-rescue:C3216X7R1H225K160AE-C3216X7R1H225K160AE C14
 U 1 1 5D36E8F9
 P 4650 3900
@@
 	6600 1950 6600 2250
 $Comp
-L IRFS7730TRLPBF:IRFS7730TRLPBF Q1
+L DSC_motor_controller-rescue:IRFS7730TRLPBF-IRFS7730TRLPBF Q1
 U 1 1 5D370686
 P 2850 1550
@@
 $EndComp
 $Comp
-L CGA6M3X7S2A475K200AB:CGA6M3X7S2A475K200AB C4
+L DSC_motor_controller-rescue:CGA6M3X7S2A475K200AB-CGA6M3X7S2A475K200AB C4
 U 1 1 5D370695
 P 3400 2250
@@
 $EndComp
 $Comp
-L CGA6M3X7S2A475K200AB:CGA6M3X7S2A475K200AB C5
+L DSC_motor_controller-rescue:CGA6M3X7S2A475K200AB-CGA6M3X7S2A475K200AB C5
 U 1 1 5D3706A4
 P 3700 2250
@@
 $EndComp
 $Comp
-L RK73H1JTTD4R70F:RK73H1JTTD4R70F R3
+L DSC_motor_controller-rescue:RK73H1JTTD4R70F-RK73H1JTTD4R70F R3
 U 1 1 5D3706B3
 P 2000 1550
@@
 $EndComp
 $Comp
-L RK73H1JTTD4R70F:RK73H1JTTD4R70F R4
+L DSC_motor_controller-rescue:RK73H1JTTD4R70F-RK73H1JTTD4R70F R4
 U 1 1 5D3706C2
 P 2050 4250
@@
 $EndComp
 $Comp
-L WSLP27261L000FEA:WSLP27261L000FEA R9
+L DSC_motor_controller-rescue:WSLP27261L000FEA-WSLP27261L000FEA R9
 U 1 1 5D3706D1
 P 1450 2000
@@
 $EndComp
 $Comp
-L AD8418ABRMZ:AD8418ABRMZ CS1
+L DSC_motor_controller-rescue:AD8418ABRMZ-AD8418ABRMZ CS1
 U 1 1 5D3706E0
 P 850 3250
@@
 $EndComp
 $Comp
-L IRFS7730TRLPBF:IRFS7730TRLPBF Q2
+L DSC_motor_controller-rescue:IRFS7730TRLPBF-IRFS7730TRLPBF Q2
 U 1 1 5D3706F1
 P 2850 4250
@@
 Connection ~ 2550 3350
 $Comp
-L C3216X7R1H225K160AE:C3216X7R1H225K160AE C13
+L DSC_motor_controller-rescue:C3216X7R1H225K160AE-C3216X7R1H225K160AE C13
 U 1 1 5D370718
 P 1700 3950
@@
 Connection ~ 650  3950
 $Comp
-L RK73H1JTTD1000F:RK73H1JTTD1000F R12
+L DSC_motor_controller-rescue:RK73H1JTTD1000F-RK73H1JTTD1000F R12
 U 1 1 5D400780
 P 2000 4850
@@
 $EndComp
 $Comp
-L GCM155R71H472KA37D:GCM155R71H472KA37D C10
+L DSC_motor_controller-rescue:GCM155R71H472KA37D-GCM155R71H472KA37D C10
 U 1 1 5D400A1D
 P 1200 5000
@@
 $EndComp
 $Comp
-L GCM155R71H472KA37D:GCM155R71H472KA37D C11
+L DSC_motor_controller-rescue:GCM155R71H472KA37D-GCM155R71H472KA37D C11
 U 1 1 5D400BA3
 P 1250 6000
@@
 $EndComp
 $Comp
-L GCM155R71H472KA37D:GCM155R71H472KA37D C12
+L DSC_motor_controller-rescue:GCM155R71H472KA37D-GCM155R71H472KA37D C12
 U 1 1 5D400C0C
 P 1250 7050
@@
 $EndComp
 $Comp
-L BLDC_4-cache:wire_pad P2
+L DSC_motor_controller-rescue:wire_pad-BLDC_4-cache P2
 U 1 1 5D465A23
 P 4600 2000
@@
 $EndComp
 $Comp
-L BLDC_4-cache:wire_pad P3
+L DSC_motor_controller-rescue:wire_pad-BLDC_4-cache P3
 U 1 1 5D465AE3
 P 8050 2050
@@
 $EndComp
 $Comp
-L BLDC_4-cache:wire_pad P1
+L DSC_motor_controller-rescue:wire_pad-BLDC_4-cache P1
 U 1 1 5D465ECF
 P 1050 2050
@@
 $EndComp
 $Comp
-L BLDC_4-cache:wire_pad P5
+L DSC_motor_controller-rescue:wire_pad-BLDC_4-cache P5
 U 1 1 5D4671C6
 P 10550 5200
@@
 $EndComp
 $Comp
-L NCP18XH103F03RB:NCP18XH103F03RB RTEMP1
+L DSC_motor_controller-rescue:NCP18XH103F03RB-NCP18XH103F03RB RTEMP1
 U 1 1 5D46A74B
 P 5000 5700
@@
 $EndComp
 $Comp
-L C3216X7R1H225K160AE:C3216X7R1H225K160AE C16
+L DSC_motor_controller-rescue:C3216X7R1H225K160AE-C3216X7R1H225K160AE C16
 U 1 1 5D46AA12
 P 4800 6600
@@
 $EndComp
 $Comp
-L RK73H1JTTD1002F:RK73H1JTTD1002F R15
+L DSC_motor_controller-rescue:RK73H1JTTD1002F-RK73H1JTTD1002F R15
 U 1 1 5D46B47E
 P 5250 6550
@@
 	5000 5550 5000 5700
 $Comp
-L RK73H1JTTD1000F:RK73H1JTTD1000F R13
+L DSC_motor_controller-rescue:RK73H1JTTD1000F-RK73H1JTTD1000F R13
 U 1 1 5D4BAFEC
 P 2050 5800
@@
 $EndComp
 $Comp
-L RK73H1JTTD1000F:RK73H1JTTD1000F R14
+L DSC_motor_controller-rescue:RK73H1JTTD1000F-RK73H1JTTD1000F R14
 U 1 1 5D4BFC80
 P 2050 6800
@@
 	7500 6150 7300 6150
 $Comp
-L BLDC_4-cache:wire_pad P4
+L DSC_motor_controller-rescue:wire_pad-BLDC_4-cache P4
 U 1 1 5D466A1B
 P 10350 700
