File: kicad_files/DSC_motor_controller.kicad_pcb (KiCad board)
At the start: 4 copper layers, 103.3 x 107.8 mm, 102 parts, among them P1 PH_A, P2 PH_B, P3 PH_C, P4 SUPPLY, P5 GND, Q1 IRFS7730TRLPBF, Q2 IRFS7730TRLPBF, Q3 IRFS7730TRLPBF, Q4 IRFS7730TRLPBF, Q5 IRFS7730TRLPBF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

Commit message: updated all files
Parts:
- added REF**: MountingHole_4.3mm_M4, MountingHole:MountingHole_4.3mm_M4, F.Cu at (62.8, 201.5)
- added REF**: MountingHole_4.3mm_M4, MountingHole:MountingHole_4.3mm_M4, F.Cu at (156.8, 201.7)
- added REF**: MountingHole_4.3mm_M4, MountingHole:MountingHole_4.3mm_M4, F.Cu at (103.7, 103.0)
- added REF**: MountingHole_4.3mm_M4, MountingHole:MountingHole_4.3mm_M4, F.Cu at (62.9, 131.8)
Routing:
- net /Motor_Driver/SH_A: track 48.7 -> 48.1 mm
Changed lines of the file:
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@@
     (thickness 1.6)
     (drawings 27)
-    (tracks 952)
+    (tracks 951)
     (zones 0)
-    (modules 102)
+    (modules 106)
     (nets 151)
   )
@@
   (layers
     (0 F.Cu signal)
-    (1 In1.Cu power hide)
-    (2 In2.Cu power hide)
-    (31 B.Cu signal hide)
-    (32 B.Adhes user hide)
-    (33 F.Adhes user hide)
-    (34 B.Paste user hide)
-    (35 F.Paste user hide)
-    (36 B.SilkS user hide)
-    (37 F.SilkS user hide)
-    (38 B.Mask user hide)
-    (39 F.Mask user hide)
-    (40 Dwgs.User user hide)
-    (41 Cmts.User user hide)
-    (42 Eco1.User user hide)
-    (43 Eco2.User user hide)
+    (1 In1.Cu power)
+    (2 In2.Cu power)
+    (31 B.Cu signal)
+    (32 B.Adhes user)
+    (33 F.Adhes user)
+    (34 B.Paste user)
+    (35 F.Paste user)
+    (36 B.SilkS user)
+    (37 F.SilkS user)
+    (38 B.Mask user)
+    (39 F.Mask user)
+    (40 Dwgs.User user)
+    (41 Cmts.User user)
+    (42 Eco1.User user)
+    (43 Eco2.User user)
     (44 Edge.Cuts user)
-    (45 Margin user hide)
-    (46 B.CrtYd user hide)
-    (47 F.CrtYd user hide)
-    (48 B.Fab user hide)
-    (49 F.Fab user hide)
+    (45 Margin user)
+    (46 B.CrtYd user)
+    (47 F.CrtYd user)
+    (48 B.Fab user)
+    (49 F.Fab user)
   )
   (setup
@@
     (add_net /Motor_Driver/PWM_C_H)
     (add_net /Motor_Driver/PWM_C_L)
+    (add_net /Motor_Driver/SH_A)
+    (add_net /Motor_Driver/SH_B)
+    (add_net /Motor_Driver/SH_C)
     (add_net /Motor_Driver/Volt_A)
     (add_net /Motor_Driver/Volt_B)
@@
     (uvia_dia 0.3)
     (uvia_drill 0.1)
-    (add_net /Motor_Driver/SH_A)
-    (add_net /Motor_Driver/SH_B)
-    (add_net /Motor_Driver/SH_C)
     (add_net "Net-(P1-Pad1)")
     (add_net "Net-(P2-Pad1)")
@@
     (add_net SUPPLY)
   )
+  (module MountingHole:MountingHole_4.3mm_M4 (layer F.Cu)
+    (at 62.775 201.525)
+    (descr "Mounting Hole 4.3mm, no annular, M4")
+    (tags "mounting hole 4.3mm no annular m4")
+    (attr virtual)
+    (fp_text reference REF** (at 0 -5.3) (layer F.SilkS)
+      (effects (font (size 1 1) (thickness 0.15)))
+    )
+    (fp_text value MountingHole_4.3mm_M4 (at 0 5.3) (layer F.Fab)
+      (effects (font (size 1 1) (thickness 0.15)))
+    )
+    (fp_text user %R (at 0.3 0) (layer F.Fab)
+      (effects (font (size 1 1) (thickness 0.15)))
+    )
+    (fp_circle (center 0 0) (end 4.3 0) (layer Cmts.User) (width 0.15))
+    (fp_circle (center 0 0) (end 4.55 0) (layer F.CrtYd) (width 0.05))
+    (pad 1 np_thru_hole circle (at 0 0) (size 4.3 4.3) (drill 4.3) (layers *.Cu *.Mask))
+  )
+  (module MountingHole:MountingHole_4.3mm_M4 (layer F.Cu)
+    (at 156.75 201.65)
+    (descr "Mounting Hole 4.3mm, no annular, M4")
+    (tags "mounting hole 4.3mm no annular m4")
+    (attr virtual)
+    (fp_text reference REF** (at 0 -5.3) (layer F.SilkS)
+      (effects (font (size 1 1) (thickness 0.15)))
+    )
+    (fp_text value MountingHole_4.3mm_M4 (at 0 5.3) (layer F.Fab)
+      (effects (font (size 1 1) (thickness 0.15)))
+    )
+    (fp_circle (center 0 0) (end 4.55 0) (layer F.CrtYd) (width 0.05))
+    (fp_circle (center 0 0) (end 4.3 0) (layer Cmts.User) (width 0.15))
+    (fp_text user %R (at 0.3 0) (layer F.Fab)
+      (effects (font (size 1 1) (thickness 0.15)))
+    )
+    (pad 1 np_thru_hole circle (at 0 0) (size 4.3 4.3) (drill 4.3) (layers *.Cu *.Mask))
+  )
+  (module MountingHole:MountingHole_4.3mm_M4 (layer F.Cu)
+    (at 103.675 102.975)
+    (descr "Mounting Hole 4.3mm, no annular, M4")
+    (tags "mounting hole 4.3mm no annular m4")
+    (attr virtual)
+    (fp_text reference REF** (at 0 -5.3) (layer F.SilkS)
+      (effects (font (size 1 1) (thickness 0.15)))
+    )
+    (fp_text value MountingHole_4.3mm_M4 (at 0 5.3) (layer F.Fab)
+      (effects (font (size 1 1) (thickness 0.15)))
+    )
+    (fp_text user %R (at 0.3 0) (layer F.Fab)
+      (effects (font (size 1 1) (thickness 0.15)))
+    )
+    (fp_circle (center 0 0) (end 4.3 0) (layer Cmts.User) (width 0.15))
+    (fp_circle (center 0 0) (end 4.55 0) (layer F.CrtYd) (width 0.05))
+    (pad 1 np_thru_hole circle (at 0 0) (size 4.3 4.3) (drill 4.3) (layers *.Cu *.Mask))
+  )
   (module "IRFS7730TRLPBF:D2PAK(TO-263AB)" (layer F.Cu)
     (at 139.954 157.48 180)
@@
     )
   )
+  (module MountingHole:MountingHole_4.3mm_M4 (layer F.Cu)
+    (at 62.925 131.8)
+    (descr "Mounting Hole 4.3mm, no annular, M4")
+    (tags "mounting hole 4.3mm no annular m4")
+    (attr virtual)
+    (fp_text reference REF** (at 0 -5.3) (layer F.SilkS)
+      (effects (font (size 1 1) (thickness 0.15)))
+    )
+    (fp_text value MountingHole_4.3mm_M4 (at 0 5.3) (layer F.Fab)
+      (effects (font (size 1 1) (thickness 0.15)))
+    )
+    (fp_circle (center 0 0) (end 4.55 0) (layer F.CrtYd) (width 0.05))
+    (fp_circle (center 0 0) (end 4.3 0) (layer Cmts.User) (width 0.15))
+    (fp_text user %R (at 0.3 0) (layer F.Fab)
+      (effects (font (size 1 1) (thickness 0.15)))
+    )
+    (pad 1 np_thru_hole circle (at 0 0) (size 4.3 4.3) (drill 4.3) (layers *.Cu *.Mask))
+  )
   (gr_line (start 67.564 126.873) (end 58.166 126.873) (layer Edge.Cuts) (width 0.03))
   (gr_line (start 67.564 133.35) (end 67.564 126.873) (layer Edge.Cuts) (width 0.03))
@@
   (via (at 96.52 187.706) (size 0.8) (drill 0.4) (layers F.Cu B.Cu) (net 1))
   (segment (start 97.2185 188.4045) (end 96.52 187.706) (width 0.25) (layer F.Cu) (net 1))
-  (segment (start 85.1905 178.912) (end 84.7635 178.485) (width 0.25) (layer F.Cu) (net 150))
-  (segment (start 84.7635 178.485) (end 84.7635 178.085) (width 0.25) (layer F.Cu) (net 150) (status 20))
-  (segment (start 86.868 178.912) (end 85.1905 178.912) (width 0.25) (layer F.Cu) (net 150) (status 10))
   (segment (start 110.82 148.312) (end 110.034 149.098) (width 0.25) (layer F.Cu) (net 2) (status 30))
   (segment (start 110.82 145.542) (end 110.82 148.312) (width 0.25) (layer F.Cu) (net 2) (status 30))
@@
   (via (at 149.479 160.401) (size 1.524) (drill 0.762) (layers F.Cu B.Cu) (net 20))
   (via (at 149.606 134.239) (size 1.524) (drill 0.762) (layers F.Cu B.Cu) (net 21))
-  (segment (start 120.142 155.693) (end 120.142 157.48) (width 0.635) (layer B.Cu) (net 21))
-  (segment (start 142.367 137.668) (end 138.167 137.668) (width 0.635) (layer B.Cu) (net 21) (status 10))
-  (segment (start 138.167 137.668) (end 120.142 155.693) (width 0.635) (layer B.Cu) (net 21))
-  (via (at 120.142 157.48) (size 0.8) (drill 0.4) (layers F.Cu B.Cu) (net 21))
-  (segment (start 120.142 157.48) (end 120.142 162.698002) (width 0.635) (layer F.Cu) (net 21))
-  (segment (start 120.142 162.698002) (end 116.216002 166.624) (width 0.25) (layer F.Cu) (net 21))
-  (segment (start 113.764 166.652) (end 111.440327 166.652) (width 0.25) (layer F.Cu) (net 21) (status 20))
-  (segment (start 113.792 166.624) (end 113.764 166.652) (width 0.635) (layer F.Cu) (net 21))
-  (segment (start 115.982 166.168) (end 115.526 166.624) (width 0.635) (layer F.Cu) (net 21))
-  (segment (start 115.982 165.608) (end 115.982 166.168) (width 0.635) (layer F.Cu) (net 21) (status 10))
-  (segment (start 116.216002 166.624) (end 113.792 166.624) (width 0.635) (layer F.Cu) (net 21))
-  (segment (start 114.3 166.624) (end 113.792 166.624) (width 0.635) (layer F.Cu) (net 21))
   (via (at 149.733 129.413) (size 1.524) (drill 0.762) (layers F.Cu B.Cu) (net 21))
   (via (at 151.384 129.413) (size 1.524) (drill 0.762) (layers F.Cu B.Cu) (net 21))
@@
   (via (at 149.606 136.017) (size 1.524) (drill 0.762) (layers F.Cu B.Cu) (net 21))
   (via (at 149.606 137.668) (size 1.524) (drill 0.762) (layers F.Cu B.Cu) (net 21))
+  (segment (start 120.142 157.48) (end 120.142 162.698002) (width 0.25) (layer F.Cu) (net 21))
+  (via (at 120.142 157.48) (size 0.8) (drill 0.4) (layers F.Cu B.Cu) (net 21))
+  (segment (start 138.167 137.668) (end 120.142 155.693) (width 0.635) (layer B.Cu) (net 21))
+  (segment (start 142.367 137.668) (end 138.167 137.668) (width 0.635) (layer B.Cu) (net 21) (status 10))
+  (segment (start 120.142 155.693) (end 120.142 157.48) (width 0.635) (layer B.Cu) (net 21))
+  (segment (start 120.142 162.698002) (end 116.216002 166.624) (width 0.25) (layer F.Cu) (net 21))
+  (segment (start 116.216002 166.402002) (end 116.216002 166.624) (width 0.25) (layer F.Cu) (net 21))
+  (segment (start 115.982 166.168) (end 116.216002 166.402002) (width 0.25) (layer F.Cu) (net 21))
+  (segment (start 115.982 165.608) (end 115.982 166.168) (width 0.25) (layer F.Cu) (net 21))
+  (segment (start 116.188002 166.652) (end 116.216002 166.624) (width 0.25) (layer F.Cu) (net 21))
+  (segment (start 111.440327 166.652) (end 116.188002 166.652) (width 0.25) (layer F.Cu) (net 21))
   (segment (start 115.062 165.598) (end 115.062 165.608) (width 0.25) (layer F.Cu) (net 22) (status 30))
   (segment (start 114.119499 164.655499) (end 115.062 165.598) (width 0.25) (layer F.Cu) (net 22) (status 20))
@@
   (segment (start 102.016 166.624) (end 101.092 165.7) (width 0.25) (layer B.Cu) (net 149) (status 20))
   (segment (start 102.616 166.624) (end 102.016 166.624) (width 0.25) (layer B.Cu) (net 149))
+  (segment (start 85.1905 178.912) (end 84.7635 178.485) (width 0.25) (layer F.Cu) (net 150))
+  (segment (start 84.7635 178.485) (end 84.7635 178.085) (width 0.25) (layer F.Cu) (net 150) (status 20))
+  (segment (start 86.868 178.912) (end 85.1905 178.912) (width 0.25) (layer F.Cu) (net 150) (status 10))
   (zone (net 140) (net_name "Net-(P3-Pad1)") (layer B.Cu) (hatch edge 0.508)
     (priority 1)
