File: kicad_files/Forward_acceleration_board/power.sch (KiCad schematic (older format))
At the start: 3 parts

Commit message: reogranized file locations, improved DSC controller pcb with edged margin on edges and rounded corners.  Completed Acceleration control board schematic
Parts:
- C1, C2: footprint CAPC1005X55N -> GRM155C91C105ME11J:CAPC1005X55N
- Reg1: footprint SOT230P700X180-4N -> TC2117-3.3VDBTR:SOT230P700X180-4N
Changed lines of the file:
@@
 $Descr A4 11693 8268
 encoding utf-8
-Sheet 4 4
+Sheet 4 6
 Title ""
 Date ""
@@
 F 0 "Reg1" H 5150 3400 50  0000 C CNN
 F 1 "TC2117" H 5150 3000 50  0000 C CNN
-F 2 "SOT230P700X180-4N" H 5650 3350 50  0001 L CNN
+F 2 "TC2117-3.3VDBTR:SOT230P700X180-4N" H 5650 3350 50  0001 L CNN
 F 3 "https://componentsearchengine.com/Datasheets/2/TC2117-3.3VDBTR.pdf" H 5650 3250 50  0001 L CNN
 F 4 "Microchip TC2117-3.3VDBTR, LDO Voltage Regulator, 800mA, 3.3 V +/-0.5%, 2.7  6 Vin, 3-Pin SOT-223" H 5650 3150 50  0001 L CNN "Description"
@@
 F 0 "C2" V 6504 3628 50  0000 L CNN
 F 1 "1u" V 6595 3628 50  0000 L CNN
-F 2 "CAPC1005X55N" H 6650 3550 50  0001 L CNN
+F 2 "GRM155C91C105ME11J:CAPC1005X55N" H 6650 3550 50  0001 L CNN
 F 3 "http://www.murata.com/~/media/webrenewal/support/library/catalog/products/capacitor/mlcc/c02e.pdf" H 6650 3450 50  0001 L CNN
 F 4 "Multilayer Ceramic Capacitors MLCC - SMD/SMT" H 6650 3350 50  0001 L CNN "Description"
@@
 F 0 "C1" V 4546 3772 50  0000 R CNN
 F 1 "1u" V 4455 3772 50  0000 R CNN
-F 2 "CAPC1005X55N" H 4600 3950 50  0001 L CNN
+F 2 "GRM155C91C105ME11J:CAPC1005X55N" H 4600 3950 50  0001 L CNN
 F 3 "http://www.murata.com/~/media/webrenewal/support/library/catalog/products/capacitor/mlcc/c02e.pdf" H 4600 3850 50  0001 L CNN
 F 4 "Multilayer Ceramic Capacitors MLCC - SMD/SMT" H 4600 3750 50  0001 L CNN "Description"
@@
 NoConn ~ 5800 3350
 $Comp
-L power:GND #PWR?
+L power:GND #PWR0135
 U 1 1 5D8DABF4
 P 6300 4100
-F 0 "#PWR?" H 6300 3850 50  0001 C CNN
+F 0 "#PWR0135" H 6300 3850 50  0001 C CNN
 F 1 "GND" H 6305 3927 50  0000 C CNN
 F 2 "" H 6300 4100 50  0001 C CNN
@@
 	4500 3900 4500 3350
 $Comp
-L power:GND #PWR?
+L power:GND #PWR0136
 U 1 1 5D8DAFBB
 P 4250 3250
-F 0 "#PWR?" H 4250 3000 50  0001 C CNN
+F 0 "#PWR0136" H 4250 3000 50  0001 C CNN
 F 1 "GND" H 4255 3077 50  0000 C CNN
 F 2 "" H 4250 3250 50  0001 C CNN
@@
 Connection ~ 4250 3250
 $Comp
-L power:+3.3V #PWR?
+L power:+3.3V #PWR0137
 U 1 1 5D8DB052
 P 4350 3900
-F 0 "#PWR?" H 4350 3750 50  0001 C CNN
+F 0 "#PWR0137" H 4350 3750 50  0001 C CNN
 F 1 "+3.3V" H 4365 4073 50  0000 C CNN
 F 2 "" H 4350 3900 50  0001 C CNN
@@
 	4350 3900 4500 3900
 $Comp
-L power:+5V #PWR?
+L power:+5V #PWR0138
 U 1 1 5D8DB134
 P 6300 3250
-F 0 "#PWR?" H 6300 3100 50  0001 C CNN
+F 0 "#PWR0138" H 6300 3100 50  0001 C CNN
 F 1 "+5V" H 6315 3423 50  0000 C CNN
 F 2 "" H 6300 3250 50  0001 C CNN
